File: cave-phone-mc34118.kicad_sch (KiCad schematic)
At the start: 0 parts

Commit message: Reference schematics (from the datasheet)
Parts:
- added C? (x4): 2µF, symbol Device:C
- added C? (x2): 47µF, symbol Device:C_Polarized
- added C?: 0,01µF, symbol Device:C
- added C? (x3): 0,05µF, symbol Device:C
- added C? (x7): 0,1µF, symbol Device:C
- added C?: 0,2µF, symbol Device:C
- added C?: 20µF, symbol Device:C_Polarized
- added C?: 270pF, symbol Device:C
- added C? (x2): 4700pF, symbol Device:C
- added C?: 5,0µF, symbol Device:C
- added C?: 200pF, symbol Device:C
- added C?: 0,02µF, symbol Device:C
- added LS?: Speaker, symbol Device:Speaker
- added MK?: Microphone_Condenser, symbol Device:Microphone_Condenser
- added R?: 620, symbol Device:R
- added R?: 330, symbol Device:R
- added R? (x2): 100K, symbol Device:R
- added R?: 220K, symbol Device:R
- added R?: 180K, symbol Device:R
- added R? (x5): 10K, symbol Device:R
- added R?: 110K, symbol Device:R
- added R? (x3): 5,1K, symbol Device:R
- added R?: 1K, symbol Device:R
- added R?: 9,1K, symbol Device:R
- added R?: 420, symbol Device:R
- added R?: 56K, symbol Device:R
- added R?: 120K, symbol Device:R
- added RV?: 20K, symbol Device:R_Potentiometer
- added SW? (x2): SW_SPST, symbol Switch:SW_SPST
- added T?: Transformer_1P_1S, symbol Device:Transformer_1P_1S
- added U?: MC34118, Package_SO:SSOP-28_5.3x10.2mm_P0.65mm, symbol cave-phone:MC34118
- added U?: MC34119P, Package_DIP:DIP-8_W7.62mm, symbol cave-phone:MC34119P
Connections:
- new net: C?.2, U?.19 (RLO2)
- new net: C?.1, R?.2, U?.16 (CPT)
- new net: C?.1, C?.1, R?.1, R?.1, T?.1 (AA)
- new net: C?.2, T?.2 (AB), U?.5 (HTO+)
- new net: C?.1, C?.1, R?.1, U?.1 (FO)
- new net: C?.1, C?.2, R?.1, R?.2, U?.10 (MCO)
- new net: C?.2, R?.1, R?.2, U?.11 (MCI)
- new net: SW?.2 (B), U?.12 (MUT)
- new net: RV?.2, U?.13 (VLC)
- new net: C?.2, R?.2, U?.14 (CT)
- new net: C?.1, U?.17 (TLI2)
- new net: C?.2, U?.18 (TLO2)
- new net: C?.2, R?.2, U?.2 (FI)
- new net: C?.2, U?.20 (RLI2)
- new net: C?.2, U?.21 (RXI)
- new net: C?.2, U?.22 (RXO)
- new net: R?.1, U?.23 (TLI1)
- new net: C?.2, U?.24 (TLO1)
- new net: C?.2, U?.25 (RLO1)
- new net: R?.2, U?.26 (RLI1)
- new net: C?.2, R?.2, U?.27 (CPR)
- new net: SW?.1 (A), U?.1 (CD), U?.3 (CD)
- new net: C?.1, C?.2, R?.1, R?.2, U?.6 (HTO-)
- new net: C?.2, R?.2, U?.7 (HTI1)
- new net: R?.1, U?.8 (TXO)
- new net: C?.1, U?.9 (TXI)
- new net: C?.2, R?.1, R?.2, U?.4 (Vin)
- new net: C?.1, LS?.2, R?.1, R?.1, U?.5 (Vo1)
- new net: LS?.1, U?.8 (Vo2)
- new net: R?.2, RV?.1
- new net: C?.2, R?.1 (x2)
- new net: C?.1, C?.2, MK?.2 (+), R?.1
- new net: C?.1, R?.1, R?.2
- new net: C?.1, R?.2 (x4)
- new net: C?.2, R?.2 (x2)
- new net: C?.1, C?.2, R?.2
- new net GND: C?.1, C?.1, C?.1, C?.1, C?.1, C?.1, C?.1, MK?.1 (-), R?.1, U?.28 (GND), U?.7 (GND)
- new net VB: C?.2, C?.2, R?.1, R?.1, RV?.3, U?.15 (VB), U?.3 (FC1)
- new net VCC: C?.1, C?.2, R?.1, R?.1, R?.2, SW?.1 (A), SW?.2 (B), U?.4 (VCC), U?.6 (Vcc)
Other:
- note added: "Enable"
- note added: "Mute"
